Commit message: Working implementation of the spawning with sensor plugins and initial control

File: waver_description/urdf/imu.xacro (robot description, xacro)
@@ -28,5 +28,5 @@
         <child link="imu_link" />
     </joint>
-    <gazebo reference="imu_link">
+    <!-- <gazebo reference="imu_link">
         <material>Gazebo/Orange</material>
         <gravity>true</gravity>
@@ -36,5 +36,5 @@
             <visualize>true</visualize>
             <topic>imu</topic>
-            <!-- <plugin filename="libgazebo_ros_imu_sensor.so" name="imu_plugin">
+            <plugin filename="libgazebo_ros_imu_sensor.so" name="imu_plugin">
                 <topicName>imu</topicName>
                 <bodyName>imu_link</bodyName>
@@ -45,7 +45,7 @@
                 <frameName>imu_link</frameName>
                 <initialOrientationAsReference>false</initialOrientationAsReference>
-            </plugin> -->
+            </plugin>
             <pose>0 0 0 0 0 0</pose>
         </sensor>
-    </gazebo>
+    </gazebo> -->
 </robot>

File: waver_description/urdf/lidar.xacro (robot description, xacro)
@@ -29,35 +29,3 @@
         <child link="ldlidar_link" />
     </joint>
-    <gazebo reference="ldlidar_link">
-        <material>Gazebo/Black</material>
-        <sensor name="${lidar_model}" type="ray">
-            <pose>0 0 0 0 0 0</pose>
-            <visualize>false</visualize>
-            <topic>scan</topic>
-            <always_on>true</always_on>
-            <update_rate>${lidar_frequency}</update_rate>
-            <ray>
-                <scan>
-                    <horizontal>
-                        <samples>${lidar_samples}</samples>
-                        <min_angle>${lidar_min_angle}</min_angle>
-                        <max_angle>${lidar_max_angle}</max_angle>
-                    </horizontal>
-                </scan>
-                <range>
-                    <min>${lidar_min_range}</min>
-                    <max>${lidar_max_range}</max>
-                </range>
-                <noise>
-                    <type>gaussian</type>
-                    <mean>0.0</mean>
-                    <stddev>0.01</stddev>
-                </noise>
-            </ray>
-            <!-- <plugin name="lidar_controller" filename="libgazebo_ros_laser.so">
-                <topicName>scan</topicName>
-                <frameName>ldlidar_link</frameName>
-            </plugin> -->
-        </sensor>
-    </gazebo>
 </robot>

File: waver_description/urdf/util.xacro (robot description, xacro)
@@ -90,6 +90,6 @@
     <xacro:property name="position_wbr_joint" value="${-pos_y_wbr} ${pos_x_wbr} ${pos_z_wbr}"/>
     <!-- Lidar specifications -->
-    <xacro:property name="mass_lidar" value="0.05" />
-    <xacro:property name="lidar_model" value="HLS-LFCD-LDS" />
+    <xacro:property name="mass_lidar" value="0.045" />
+    <xacro:property name="lidar_model" value="D500" />
     <xacro:property name="lidar_link" value="lidar_link" />
     <xacro:property name="lidar_samples" value="720" />
@@ -98,4 +98,5 @@
     <xacro:property name="lidar_max_angle" value="${pi}" />
     <xacro:property name="lidar_min_angle" value="-${pi}" />
+    <xacro:property name="lidar_resolution" value="1" />
     <xacro:property name="lidar_frequency" value="10" />
     <xacro:property name="lidar_transform" value="0 0 0 0 0 0" />

File: waver_description/urdf/waver.gazebo.xacro (robot description, xacro)
@@ -1,88 +1,167 @@
 <?xml version="1.0"?>
 <robot xmlns:xacro="http://www.ros.org/wiki/xacro" name="waver_gazebo">
-  <xacro:include filename="$(find waver_description)/urdf/util.xacro" />
-  <gazebo reference="base_link">
-    <mu1>0.2</mu1>
-    <mu2>0.2</mu2>
-    <selfCollide>false</selfCollide>
-    <material>Gazebo/DarkGrey</material>
-  </gazebo>
-  <gazebo reference="top_shell_link">
-    <mu1>0.2</mu1>
-    <mu2>0.2</mu2>
-    <selfCollide>false</selfCollide>
-    <material>Gazebo/DarkGrey</material>
-  </gazebo>
-  <gazebo reference="accessories_link">
-    <mu1>0.2</mu1>
-    <mu2>0.2</mu2>
-    <selfCollide>false</selfCollide>
-    <material>Gazebo/Black</material>
-  </gazebo>
-  <gazebo reference="accessories1_link">
-    <mu1>0.2</mu1>
-    <mu2>0.2</mu2>
-    <selfCollide>false</selfCollide>
-    <material>Gazebo/Black</material>
-  </gazebo>
-  <gazebo reference="imu_link">
-    <mu1>0.2</mu1>
-    <mu2>0.2</mu2>
-    <selfCollide>false</selfCollide>
-    <material>Gazebo/Orange</material>
-  </gazebo>
-  <gazebo reference="oled_screen_link">
-    <mu1>0.2</mu1>
-    <mu2>0.2</mu2>
-    <selfCollide>false</selfCollide>
-    <material>Gazebo/BlueGlow</material>
-  </gazebo>
-  <gazebo reference="wheel_back_left_link">
-    <mu1>0.2</mu1>
-    <mu2>0.2</mu2>
-    <selfCollide>false</selfCollide>
-    <material>Gazebo/Black</material>
-  </gazebo>
-  <gazebo reference="wheel_front_left_link">
-    <mu1>0.2</mu1>
-    <mu2>0.2</mu2>
-    <selfCollide>false</selfCollide>
-    <material>Gazebo/Black</material>
-  </gazebo>
-  <gazebo reference="wheel_front_right_link">
-    <mu1>0.2</mu1>
-    <mu2>0.2</mu2>
-    <selfCollide>false</selfCollide>
-    <material>Gazebo/Black</material>
-  </gazebo>
-  <gazebo reference="wheel_back_right_link">
-    <mu1>0.2</mu1>
-    <mu2>0.2</mu2>
-    <selfCollide>false</selfCollide>
-    <material>Gazebo/Black</material>
-  </gazebo>
-  <gazebo>
-    <!-- <plugin name="skid_steer_drive_controller" filename="libgazebo_ros_skid_steer_drive.so">
-      <robotNamespace></robotNamespace>
-      <updateRate>100.0</updateRate>
-      <leftFrontJoint>wheel_front_left_joint</leftFrontJoint>
-      <rightFrontJoint>wheel_front_right_joint</rightFrontJoint>
-      <leftRearJoint>wheel_back_left_joint</leftRearJoint>
-      <rightRearJoint>wheel_back_right_joint</rightRearJoint>
-      <wheelSeparation>${wheel_separation}</wheelSeparation>
-      <wheelDiameter>${2*wheel_radius}</wheelDiameter>
-      <torque>2</torque>
-      <commandTopic>cmd_vel</commandTopic>
-      <odometryTopic>odom</odometryTopic>
-      <odometryFrame>odom</odometryFrame>
-      <robotBaseFrame>base_footprint</robotBaseFrame>
-      <publishWheelTF>true</publishWheelTF>
-      <publishOdom>true</publishOdom>
-      <publishWheelJointState>true</publishWheelJointState>
-      <covariance_x>0.0001</covariance_x>
-      <covariance_y>0.0001</covariance_y>
-      <covariance_yaw>0.01</covariance_yaw>
-      <broadcastTF>true</broadcastTF>
-    </plugin> -->
-  </gazebo>
+  <xacro:macro name="waver_robot_gazebo">
+    <xacro:include filename="$(find waver_description)/urdf/util.xacro" />
+      <!-- =============== Gazebo =============== -->
+      <gazebo>
+        <plugin filename="gz_ros2_control-system" name="gz_ros2_control::GazeboSimROS2ControlPlugin">
+          <parameters>$(find waver_description)/config/waver_robot_sim.yaml</parameters>
+        </plugin>
+        <plugin filename="gz-sim-sensors-system" name="gz::sim::systems::Sensors">
+          <render_engine>ogre2</render_engine>
+        </plugin>
+        <plugin filename="gz-sim-imu-system" name="gz::sim::systems::Imu">
+        </plugin>
+      </gazebo>
+      <gazebo reference="ldlidar_link" >
+        <sensor name="${lidar_model}" type="gpu_lidar">
+          <gz_frame_id>ldlidar_link</gz_frame_id>
+          <topic>scan</topic>
+          <update_rate>${lidar_frequency}</update_rate>
+          <lidar>
+            <scan>
+              <horizontal>
+                <samples>${lidar_samples}</samples>
+                <resolution>${lidar_resolution}</resolution>
+                <min_angle>${lidar_min_angle}</min_angle>
+                <max_angle>${lidar_max_angle}</max_angle>
+              </horizontal>
+              <vertical>
+                <samples>1</samples>
+                <resolution>0.1</resolution>
+                <min_angle>0.0</min_angle>
+                <max_angle>0.0</max_angle>
+              </vertical>
+            </scan>
+            <range>
+              <min>${lidar_min_range}</min>
+              <max>${lidar_max_range}</max>
+              <resolution>0.01</resolution>
+            </range>
+            <frame_id>/ldlidar_link</frame_id>
+          </lidar>
+          <alwaysOn>1</alwaysOn>
+          <visualize>true</visualize>
+        </sensor>
+      </gazebo>
+      <gazebo reference="imu_link" >
+        <sensor name="imu_sensor" type="imu">
+          <gz_frame_id>imu_link</gz_frame_id>
+          <topic>imu</topic>
+          <update_rate>200</update_rate>
+          <always_on>1</always_on>
+          <visualize>true</visualize>
+        </sensor>
+      </gazebo>
+      <gazebo reference="base_link">
+        <sensor name="camera_sensor" type="camera">
+          <gz_frame_id>base_link</gz_frame_id>
+          <topic>camera/image_raw</topic>
+          <update_rate>30</update_rate>
+          <camera>
+            <horizontal_fov>1.57</horizontal_fov> <!-- 90 degrees FOV -->
+            <image>
+              <width>640</width>
+              <height>480</height>
+              <format>R8G8B8</format> <!-- RGB format -->
+            </image>
+            <clip>
+              <near>0.01</near>
+              <far>100.0</far>
+            </clip>
+            <noise>
+              <type>gaussian</type>
+              <mean>0.0</mean>
+              <stddev>0.007</stddev>
+            </noise>
+          </camera>
+          <always_on>1</always_on>
+          <visualize>true</visualize>
+        </sensor>
+      </gazebo>
+      <gazebo reference="base_link">
+        <mu1>0.2</mu1>
+        <mu2>0.2</mu2>
+        <selfCollide>false</selfCollide>
+        <material>Gazebo/DarkGrey</material>
+      </gazebo>
+      <gazebo reference="top_shell_link">
+        <mu1>0.2</mu1>
+        <mu2>0.2</mu2>
+        <selfCollide>false</selfCollide>
+        <material>Gazebo/DarkGrey</material>
+      </gazebo>
+      <gazebo reference="accessories_link">
+        <mu1>0.2</mu1>
+        <mu2>0.2</mu2>
+        <selfCollide>false</selfCollide>
+        <material>Gazebo/Black</material>
+      </gazebo>
+      <gazebo reference="accessories1_link">
+        <mu1>0.2</mu1>
+        <mu2>0.2</mu2>
+        <selfCollide>false</selfCollide>
+        <material>Gazebo/Black</material>
+      </gazebo>
+      <gazebo reference="imu_link">
+        <mu1>0.2</mu1>
+        <mu2>0.2</mu2>
+        <selfCollide>false</selfCollide>
+        <material>Gazebo/Orange</material>
+      </gazebo>
+      <gazebo reference="oled_screen_link">
+        <mu1>0.2</mu1>
+        <mu2>0.2</mu2>
+        <selfCollide>false</selfCollide>
+        <material>Gazebo/BlueGlow</material>
+      </gazebo>
+      <gazebo reference="wheel_back_left_link">
+        <mu1>0.2</mu1>
+        <mu2>0.2</mu2>
+        <selfCollide>false</selfCollide>
+        <material>Gazebo/Black</material>
+      </gazebo>
+      <gazebo reference="wheel_front_left_link">
+        <mu1>0.2</mu1>
+        <mu2>0.2</mu2>
+        <selfCollide>false</selfCollide>
+        <material>Gazebo/Black</material>
+      </gazebo>
+      <gazebo reference="wheel_front_right_link">
+        <mu1>0.2</mu1>
+        <mu2>0.2</mu2>
+        <selfCollide>false</selfCollide>
+        <material>Gazebo/Black</material>
+      </gazebo>
+      <gazebo reference="wheel_back_right_link">
+        <mu1>0.2</mu1>
+        <mu2>0.2</mu2>
+        <selfCollide>false</selfCollide>
+        <material>Gazebo/Black</material>
+      </gazebo>
+      <gazebo>
+        <!-- <plugin name="skid_steer_drive_controller" filename="libgazebo_ros_skid_steer_drive.so">
+          <robotNamespace></robotNamespace>
+          <updateRate>100.0</updateRate>
+          <leftFrontJoint>wheel_front_left_joint</leftFrontJoint>
+          <rightFrontJoint>wheel_front_right_joint</rightFrontJoint>
+          <leftRearJoint>wheel_back_left_joint</leftRearJoint>
+          <rightRearJoint>wheel_back_right_joint</rightRearJoint>
+          <wheelSeparation>${wheel_separation}</wheelSeparation>
+          <wheelDiameter>${2*wheel_radius}</wheelDiameter>
+          <torque>2</torque>
+          <commandTopic>cmd_vel</commandTopic>
+          <odometryTopic>odom</odometryTopic>
+          <odometryFrame>odom</odometryFrame>
+          <robotBaseFrame>base_footprint</robotBaseFrame>
+          <publishWheelTF>true</publishWheelTF>
+          <publishOdom>true</publishOdom>
+          <publishWheelJointState>true</publishWheelJointState>
+          <covariance_x>0.0001</covariance_x>
+          <covariance_y>0.0001</covariance_y>
+          <covariance_yaw>0.01</covariance_yaw>
+          <broadcastTF>true</broadcastTF>
+        </plugin> -->
+      </gazebo>
+  </xacro:macro>
 </robot>

File: waver_description/urdf/waver.xacro (robot description, xacro)
@@ -5,4 +5,5 @@
   <xacro:include filename="$(find waver_description)/urdf/waver.trans.xacro" />
   <xacro:include filename="$(find waver_description)/urdf/waver.gazebo.xacro" />
+  <xacro:include filename="$(find waver_description)/ros2_control/waver_robot.ros2_control.xacro" />
   <xacro:include filename="$(find waver_description)/urdf/lidar.xacro" />
   <xacro:include filename="$(find waver_description)/urdf/imu.xacro" />
@@ -240,3 +241,6 @@
     <axis xyz="0 1 0" />
   </joint>
+  <!-- Gazebo -->
+  <xacro:waver_robot_gazebo/>
+  <xacro:waver_robot_ros2_control/>
 </robot>

Commit message: Fixups

File: waver_description/urdf/imu.xacro (robot description, xacro)
@@ -28,24 +28,3 @@
         <child link="imu_link" />
     </joint>
-    <!-- <gazebo reference="imu_link">
-        <material>Gazebo/Orange</material>
-        <gravity>true</gravity>
-        <sensor name="imu_sensor" type="imu">
-            <always_on>true</always_on>
-            <update_rate>100</update_rate>
-            <visualize>true</visualize>
-            <topic>imu</topic>
-            <plugin filename="libgazebo_ros_imu_sensor.so" name="imu_plugin">
-                <topicName>imu</topicName>
-                <bodyName>imu_link</bodyName>
-                <updateRateHZ>10.0</updateRateHZ>
-                <gaussianNoise>0.0</gaussianNoise>
-                <xyzOffset>0 0 0</xyzOffset>
-                <rpyOffset>0 0 0</rpyOffset>
-                <frameName>imu_link</frameName>
-                <initialOrientationAsReference>false</initialOrientationAsReference>
-            </plugin>
-            <pose>0 0 0 0 0 0</pose>
-        </sensor>
-    </gazebo> -->
 </robot>

File: waver_description/urdf/waver.gazebo.xacro (robot description, xacro)
@@ -140,28 +140,4 @@
         <material>Gazebo/Black</material>
       </gazebo>
-      <gazebo>
-        <!-- <plugin name="skid_steer_drive_controller" filename="libgazebo_ros_skid_steer_drive.so">
-          <robotNamespace></robotNamespace>
-          <updateRate>100.0</updateRate>
-          <leftFrontJoint>wheel_front_left_joint</leftFrontJoint>
-          <rightFrontJoint>wheel_front_right_joint</rightFrontJoint>
-          <leftRearJoint>wheel_back_left_joint</leftRearJoint>
-          <rightRearJoint>wheel_back_right_joint</rightRearJoint>
-          <wheelSeparation>${wheel_separation}</wheelSeparation>
-          <wheelDiameter>${2*wheel_radius}</wheelDiameter>
-          <torque>2</torque>
-          <commandTopic>cmd_vel</commandTopic>
-          <odometryTopic>odom</odometryTopic>
-          <odometryFrame>odom</odometryFrame>
-          <robotBaseFrame>base_footprint</robotBaseFrame>
-          <publishWheelTF>true</publishWheelTF>
-          <publishOdom>true</publishOdom>
-          <publishWheelJointState>true</publishWheelJointState>
-          <covariance_x>0.0001</covariance_x>
-          <covariance_y>0.0001</covariance_y>
-          <covariance_yaw>0.01</covariance_yaw>
-          <broadcastTF>true</broadcastTF>
-        </plugin> -->
-      </gazebo>
   </xacro:macro>
 </robot>
