Commit message: Added waver_navigation

File: waver_description/urdf/util.xacro (robot description, xacro)
@@ -99,5 +99,5 @@
     <xacro:property name="lidar_min_angle" value="-${pi}" />
     <xacro:property name="lidar_resolution" value="1" />
-    <xacro:property name="lidar_frequency" value="10" />
+    <xacro:property name="lidar_frequency" value="50" />
     <xacro:property name="lidar_transform" value="0 0 0 0 0 0" />
 </robot>

File: waver_description/urdf/waver.gazebo.xacro (robot description, xacro)
@@ -10,21 +10,21 @@
           <right_joint>wheel_front_right_joint</right_joint>
           <right_joint>wheel_back_right_joint</right_joint>
-          <wheel_separation>0.156</wheel_separation>
-          <wheel_radius>0.026</wheel_radius>
+          <wheel_separation>123e-3</wheel_separation>
+          <wheel_radius>40.6e-3"</wheel_radius>
           <!-- Control gains and limits (optional) -->
-          <max_velocity>3.0</max_velocity>                <!-- Max linear velocity in m/s -->
+          <max_velocity>1.25</max_velocity>                <!-- Max linear velocity in m/s -->
           <max_linear_acceleration>1</max_linear_acceleration>
           <min_linear_acceleration>-1</min_linear_acceleration>
           <max_angular_acceleration>2</max_angular_acceleration>
           <min_angular_acceleration>-2</min_angular_acceleration>
-          <max_linear_velocity>0.5</max_linear_velocity>
+          <!-- <max_linear_velocity>0.5</max_linear_velocity>
           <min_linear_velocity>-0.5</min_linear_velocity>
           <max_angular_velocity>1</max_angular_velocity>
-          <min_angular_velocity>-1</min_angular_velocity>
+          <min_angular_velocity>-1</min_angular_velocity> -->
           <topic>cmd_vel</topic>
           <odom_topic>odom</odom_topic>
           <frame_id>odom</frame_id>
           <child_frame_id>base_footprint</child_frame_id>
-          <odom_publisher_frequency>30</odom_publisher_frequency>
+          <odom_publisher_frequency>50</odom_publisher_frequency>
           <tf_topic>/tf</tf_topic>
         </plugin>
@@ -56,10 +56,10 @@
                 <max_angle>${lidar_max_angle}</max_angle>
               </horizontal>
-              <vertical>
+              <!-- <vertical>
                 <samples>1</samples>
                 <resolution>0.1</resolution>
                 <min_angle>0.0</min_angle>
                 <max_angle>0.0</max_angle>
-              </vertical>
+              </vertical> -->
             </scan>
             <range>

Commit message: Increased wheel separation fixing the odom

File: waver_description/urdf/util.xacro (robot description, xacro)
@@ -99,5 +99,5 @@
     <xacro:property name="lidar_min_angle" value="-${pi}" />
     <xacro:property name="lidar_resolution" value="1" />
-    <xacro:property name="lidar_frequency" value="50" />
+    <xacro:property name="lidar_frequency" value="10" />
     <xacro:property name="lidar_transform" value="0 0 0 0 0 0" />
 </robot>

File: waver_description/urdf/waver.gazebo.xacro (robot description, xacro)
@@ -10,5 +10,5 @@
           <right_joint>wheel_front_right_joint</right_joint>
           <right_joint>wheel_back_right_joint</right_joint>
-          <wheel_separation>123e-3</wheel_separation>
+          <wheel_separation>0.188</wheel_separation>
           <wheel_radius>40.6e-3"</wheel_radius>
           <!-- Control gains and limits (optional) -->
@@ -26,5 +26,5 @@
           <frame_id>odom</frame_id>
           <child_frame_id>base_footprint</child_frame_id>
-          <odom_publisher_frequency>50</odom_publisher_frequency>
+          <odom_publisher_frequency>30</odom_publisher_frequency>
           <tf_topic>/tf</tf_topic>
         </plugin>
@@ -68,5 +68,5 @@
               <resolution>0.01</resolution>
             </range>
-            <frame_id>/ldlidar_link</frame_id>
+            <frame_id>ldlidar_link</frame_id>
           </lidar>
           <alwaysOn>1</alwaysOn>
